File: my-project.kicad_pcb (KiCad board)
At the start: 2 copper layers, 81.3 x 40.1 mm, 63 parts, among them J1 USB_C_Receptacle_USB2.0, J2 Conn_01x04, J3 Conn_01x02, J4 Conn_01x19, J5 Conn_01x20, J6 Conn_01x02, J7 Conn_01x03, Q1 Q_PMOS_GSD, SW1 SW_Push, SW2 SW_Push, SW3 SW_Push, SW4 SW_Push, U1 CH340E, U2 TJA1051T-3, U3 HX9193, U4 STM32F103C8Tx, U5 AD8400ARZ50, Y1 Crystal_GND24

Commit message: Add files via upload
Parts:
- moved LED2 3.83 mm to (192.7, 67.7), turned to 180 degrees
- moved R7 3.78 mm to (189.2, 69.5)
- moved LED1 3.48 mm to (192.6, 69.5), turned to 180 degrees
- renumbered D2 to LED1, D3 to LED2
Routing:
- net +3.3V: track 306.9 -> 298.3 mm, vias 16 -> 15
- net /STM32_MinimumSystem/PB3: track 18.9 -> 24.2 mm
- net /STM32_MinimumSystem/PA15: track 19.7 -> 24.4 mm
Other:
- board text added: "5V"
- board text added: "A0"
- board text added: "A1"
- board text added: "A10"
- board text added: "A11"
- board text added: "A12"
- board text added: "A15"
- board text added: "A2"
- board text added: "A3"
- board text added: "A4"
- board text added: "A5"
- board text added: "A6"
- board text added: "A7"
- board text added: "A8"
- board text added: "A9"
- board text added: "B0"
- board text added: "B1"
- board text added: "B10"
- board text added: "B11"
- board text added: "B12"
- board text added: "B13"
- board text added: "B14"
- board text added: "B15"
- board text added: "B2"
- board text added: "B3"
- board text added: "B4"
- board text added: "B5"
- board text added: "B6"
- board text added: "B7"
- board text added: "B8"
- board text added: "B9"
- board text added: "BOOT0"
- board text added: "BT0"
- board text added: "C13"
- board text added: "C14"
- board text added: "C15"
- board text added: "PA0"
- board text added: "PA1"
- board text added: "PA10"
- board text added: "PA11"
- board text added: "PA12"
- board text added: "PA15"
- board text added: "PA2"
- board text added: "PA3"
- board text added: "PA4"
- board text added: "PA5"
- board text added: "PA6"
- board text added: "PA7"
- board text added: "PA8"
- board text added: "PA9"
- board text added: "PB0"
- board text added: "PB1"
- board text added: "PB10"
- board text added: "PB11"
- board text added: "PB12"
- board text added: "PB13"
- board text added: "PB14"
- board text added: "PB15"
- board text added: "PB2"
- board text added: "PB3"
- board text added: "PB4"
- board text added: "PB5"
- board text added: "PB6"
- board text added: "PB7"
- board text added: "PB8"
- board text added: "PB9"
- board text added: "PC13"
- board text added: "PC14"
- board text added: "PC15"
